File: ISS.kicad_pcb (KiCad board)
At the start: 2 copper layers, 304.9 x 129.5 mm, 131 parts, among them J2 Conn_01x08, J4 DEBUG, J5 OLED, J6 EPAPER RIBBON, M1 M.2_Key_E, U1 XC6206P332MR

Commit message: db stuff and spi pin deciding spreadsheet
Parts:
- added F1: Polyfuse, Resistor_SMD:R_0805_2012Metric, F.Cu at (50.1, 179.3)
- added J1: HRO-TYPEC-M12, Connector_USB:USB_C_Receptacle_HRO_TYPE-C-31-M-12, F.Cu at (53.8, 173.2)
- added J3: BATTERY, Connector_JST:JST_PH_S2B-PH-SM4-TB_1x02-1MP_P2.00mm_Horizontal, F.Cu at (76.1, 164.5)
- added J7: DB FFC, Connector-pat-various:100519220810EHLF, F.Cu at (64.6, 171.5)
- added J8: SPLIT, Connector-pat-various:Magnetic Pogo 4 pin, F.Cu at (59.4, 159.9)
- added MO10: MOUNTING, MountingHole:MountingHole_2.2mm_M2_Pad, F.Cu at (62.6, 177.8)
- added MO11: MOUNTING, MountingHole:MountingHole_2.2mm_M2_Pad, F.Cu at (72.6, 173.1)
- added MO9: MOUNTING, MountingHole:MountingHole_2.2mm_M2_Pad, F.Cu at (84.2, 161.8)
- added R1: 5.1k, Resistor_SMD:R_0402_1005Metric, F.Cu at (53.8, 178.9)
- added R2: 5.1k, Resistor_SMD:R_0402_1005Metric, F.Cu at (56.7, 178.9)
- added U2: SRV05-4, Package_TO_SOT_SMD:SOT-23-6, F.Cu at (68.1, 178.3)
- J2: value Conn_01x08 -> DB FFC
- moved LO1 12.8 mm to (116.0, 58.0)
Connections:
- J2 pad 3: unconnected-(J2-Pad3) -> GND
- UG2 pad 1: Net-(UG2-Pad1) -> Net-(UG1-Pad3)
- UG2 pad 3: Net-(UG1-Pad1) -> Net-(UG2-Pad3)
- UG3 pad 1: unconnected-(UG3-Pad1) -> Net-(UG2-Pad3)
- UG3 pad 3: Net-(UG2-Pad1) -> /Left/rgbin
- UG4 pad 1: Net-(UG1-Pad3) -> Net-(UG4-Pad1)
- UG4 pad 3: Net-(UG4-Pad3) -> Net-(UG1-Pad1)
- UG5 pad 1: Net-(UG4-Pad3) -> Net-(UG5-Pad1)
- UG5 pad 3: Net-(UG5-Pad3) -> Net-(UG4-Pad1)
- UG6 pad 1: Net-(UG5-Pad3) -> Net-(UG6-Pad1)
- UG6 pad 3: Net-(UG6-Pad3) -> Net-(UG5-Pad1)
- UG7 pad 1: Net-(UG6-Pad3) -> Net-(UG7-Pad1)
- UG7 pad 3: Net-(UG7-Pad3) -> Net-(UG6-Pad1)
- UG9 pad 1: Net-(UG7-Pad3) -> unconnected-(UG9-Pad1)
- UG9 pad 3: /Left/rgbin -> Net-(UG7-Pad1)
- UG9 pad 4: unconnected-(UG9-Pad4) -> Net-(R5-Pad1)
Routing:
- net GND: track 25.6 -> 28.4 mm, vias 22 -> 23
